Commit message: Gmapping configured

File: sugv_description/urdf/sugv.xacro (robot description, xacro)
@@ -1,5 +1,4 @@
 <?xml version="1.0"?>
 <robot xmlns:xacro="http://www.ros.org/wiki/xacro" name="sugv">
-	<xacro:arg name="robot_namespace" default="/" />
 	<xacro:property name="body_height" value="0.1" />
 	<xacro:property name="body_radius" value="0.2" />
@@ -12,5 +11,5 @@
 	<xacro:property name="lidar_height" value="0.04" />
 	<xacro:property name="lidar_radius" value="0.035" />
-	<link name="link_body">
+	<link name="base_link">
 		<inertial>
 			<origin xyz="0.0 0.0 0.0" rpy="0.0 0.0 0.0"/>
@@ -23,5 +22,5 @@
 			</geometry>
 			<material name="white">
-				<color rgba="1 1 1 0.1" />
+				<color rgba="1 1 1 0.5" />
 			</material>
 		</visual>
@@ -34,5 +33,5 @@
 	<link name="link_imu" />
 	<joint name="joint_imu" type="fixed">
-		<parent link="link_body"/>
+		<parent link="base_link"/>
 		<child link="link_imu"/>
 		<origin xyz="0.0 0.0 0.0" rpy="0.0 0.0 0.0"/>
@@ -47,5 +46,5 @@
 	</link>
 	<joint name="joint_lidar" type="fixed">
-		<parent link="link_body"/>
+		<parent link="base_link"/>
 		<child link="link_laser"/>
 		<origin xyz="0.0 0.0 ${body_height/2 + lidar_height/2}" rpy="0.0 0.0 0.0"/>
@@ -83,5 +82,5 @@
 		</gazebo>
 		<joint name="joint_wheel_${wheel_prefix}" type="continuous">
-			<parent link="link_body"/>
+			<parent link="base_link"/>
 			<child link="link_wheel_${wheel_prefix}"/>
 			<axis xyz="0 1 0"/>
@@ -128,5 +127,5 @@
 		</gazebo>
 		<joint name="joint_caster_${wheel_prefix}" type="fixed">
-			<parent link="link_body"/>
+			<parent link="base_link"/>
 			<child link="link_caster_${wheel_prefix}"/>
 			<axis xyz="0 1 0"/>
@@ -148,5 +147,4 @@
 	<gazebo>
 		<plugin name="gazebo_ros_control" filename="libgazebo_ros_control.so">
-			<robotNamespace>$(arg robot_namespace)</robotNamespace>
 		</plugin>
 	</gazebo>
@@ -159,6 +157,5 @@
 			<topic>__default_topic__</topic>
 			<plugin filename="libgazebo_ros_imu_sensor.so" name="imu_plugin">
-				<robotNamespace>$(arg robot_namespace)</robotNamespace>
-				<topicName>imu</topicName>
+				<topicName>sensor/imu</topicName>
 				<bodyName>link_imu</bodyName>
 				<updateRateHZ>10.0</updateRateHZ>
@@ -175,5 +172,5 @@
 		<material>Gazebo/Orange</material>
 		<sensor type="ray" name="head_rplidar_sensor">
-			<pose>0 0 0 0 0 0</pose>
+			<pose>0 0 ${body_height/2 + lidar_height/2} 0 0 0</pose>
 			<visualize>true</visualize>
 			<update_rate>40</update_rate>
@@ -199,6 +196,5 @@
 			</ray>
 			<plugin name="gazebo_ros_head_rplidar_controller" filename="libgazebo_ros_laser.so">
-				<robotNamespace>$(arg robot_namespace)</robotNamespace>
-				<topicName>scan</topicName>
+				<topicName>sensor/scan</topicName>
 				<frameName>link_laser</frameName>
 			</plugin>
